Commit message: sadasd

File: PC_user/src/Hardware/manipulator/manipulator_description/urdf/manipulator.urdf.xacro (robot description, xacro)
@@ -1,5 +1,5 @@
 <?xml version="1.0"?>
 <robot xmlns:xacro="http://ros.org/wiki/xacro">
-<xacro:macro name="prismatic_manipulator" params="prefix parent_link mesh_package xyz rpy">
+<xacro:macro name="prismatic_manipulator" params="parent_link mesh_package xyz rpy">
   <xacro:property name="scale" value="0.001 0.001 0.001"/>
   <!-- Materiales -->
@@ -11,5 +11,5 @@
   </material>
   <!-- Links -->
-  <link name="${prefix}BaseFrame_link">
+  <link name="BaseFrame_link">
     <visual>
       <geometry>
@@ -24,5 +24,5 @@
     </collision>
   </link>
-  <link name="${prefix}AxisY_link">
+  <link name="AxisY_link">
     <visual>
       <geometry>
@@ -37,5 +37,5 @@
     </collision>
   </link>
-  <link name="${prefix}AxisX_link">
+  <link name="AxisX_link">
     <visual>
       <geometry>
@@ -50,5 +50,5 @@
     </collision>
   </link>
-  <link name="${prefix}AxisZ_link">
+  <link name="AxisZ_link">
     <visual>
       <geometry>
@@ -63,5 +63,5 @@
     </collision>
   </link>
-  <link name="${prefix}ClawBase_link">
+  <link name="ClawBase_link">
     <visual>
       <geometry>
@@ -76,5 +76,5 @@
     </collision>
   </link>
-  <link name="${prefix}ClawShovelR_link">
+  <link name="ClawShovelR_link">
     <visual>
       <geometry>
@@ -89,5 +89,5 @@
     </collision>
   </link>
-  <link name="${prefix}ClawShovelL_link">
+  <link name="ClawShovelL_link">
     <visual>
       <geometry>
@@ -103,12 +103,12 @@
   </link>
   <!-- Joints -->
-  <joint name="${prefix}BaseFrame_joint" type="fixed">
+  <joint name="BaseFrame_joint" type="fixed">
     <parent link="${parent_link}"/>
-    <child link="${prefix}BaseFrame_link"/>
+    <child link="BaseFrame_link"/>
     <origin xyz="${xyz}" rpy="${rpy}"/>
   </joint>
-  <joint name="${prefix}AxisY_joint" type="prismatic">
-    <parent link="${prefix}BaseFrame_link"/>
-    <child link="${prefix}AxisY_link"/>
+  <joint name="AxisY_joint" type="prismatic">
+    <parent link="BaseFrame_link"/>
+    <child link="AxisY_link"/>
     <origin xyz="-0.00475 0.25696 0.02" rpy="0 0 0"/>
     <axis xyz="0 1 0"/>
@@ -116,7 +116,7 @@
     <dynamics damping="0.7" friction="0.1"/>
   </joint>
-  <joint name="${prefix}AxisX_joint" type="prismatic">
-    <parent link="${prefix}AxisY_link"/>
-    <child link="${prefix}AxisX_link"/>
+  <joint name="AxisX_joint" type="prismatic">
+    <parent link="AxisY_link"/>
+    <child link="AxisX_link"/>
     <origin xyz="0.02504 0.056 0.081" rpy="0 0 0"/>
     <axis xyz="1 0 0"/>
@@ -124,7 +124,7 @@
     <dynamics damping="0.5" friction="0.1"/>
   </joint>
-  <joint name="${prefix}AxisZ_joint" type="prismatic">
-    <parent link="${prefix}AxisX_link"/>
-    <child link="${prefix}AxisZ_link"/>
+  <joint name="AxisZ_joint" type="prismatic">
+    <parent link="AxisX_link"/>
+    <child link="AxisZ_link"/>
     <origin xyz="0.035 -0.05745 0.21389" rpy="0 0 0"/>
     <axis xyz="0 0 1"/>
@@ -132,12 +132,12 @@
     <dynamics damping="0.3" friction="0.05"/>
   </joint>
-  <joint name="${prefix}ClawBase_joint" type="fixed">
-    <parent link="${prefix}AxisZ_link"/>
-    <child link="${prefix}ClawBase_link"/>
+  <joint name="ClawBase_joint" type="fixed">
+    <parent link="AxisZ_link"/>
+    <child link="ClawBase_link"/>
     <origin xyz="-0.01 -0.24 0.03" rpy="0 0 0"/>
   </joint>
-  <joint name="${prefix}ClawShovelR_joint" type="prismatic">
-    <parent link="${prefix}ClawBase_link"/>
-    <child link="${prefix}ClawShovelR_link"/>
+  <joint name="ClawShovelR_joint" type="prismatic">
+    <parent link="ClawBase_link"/>
+    <child link="ClawShovelR_link"/>
     <origin xyz="-0.0357 -0.04494 -0.04010" rpy="0 0 0"/>
     <axis xyz="1 0 0"/>
@@ -145,7 +145,7 @@
     <dynamics damping="0.3" friction="0.05"/>
   </joint>
-  <joint name="${prefix}ClawShovelL_joint" type="prismatic">
-    <parent link="${prefix}ClawBase_link"/>
-    <child link="${prefix}ClawShovelL_link"/>
+  <joint name="ClawShovelL_joint" type="prismatic">
+    <parent link="ClawBase_link"/>
+    <child link="ClawShovelL_link"/>
     <origin xyz="0.0557 0.0549 -0.04010" rpy="0 0 3.141516"/>
     <axis xyz="1 0 0"/>

File: PC_user/src/Hardware/robotino/robotino_description/urdf/robotino.urdf.xacro (robot description, xacro)
@@ -122,5 +122,4 @@
   <!-- ==================== Manipulator (Prismatic) ==================== -->
   <xacro:prismatic_manipulator
-      prefix="manipulator_"
       parent_link="platform_link"
       mesh_package="manipulator_description"

Commit message: Update urdf model

File: PC_user/src/Hardware/manipulator/manipulator_description/urdf/manipulator.urdf.xacro (robot description, xacro)
@@ -102,4 +102,6 @@
     </collision>
   </link>
+  <link name="realsense_link">
+  </link>
   <!-- Joints -->
   <joint name="BaseFrame_joint" type="fixed">
@@ -137,4 +139,9 @@
     <origin xyz="-0.01 -0.24 0.03" rpy="0 0 0"/>
   </joint>
+  <joint name="realsense_joint" type="fixed">
+    <parent link="ClawBase_link"/>
+    <child link="realsense_link"/>
+    <origin xyz="0.027 -0.035 -0.018" rpy="1.5707 1.5707 0"/>
+  </joint>
   <joint name="ClawShovelR_joint" type="prismatic">
     <parent link="ClawBase_link"/>

File: PC_user/src/Hardware/robotino/robotino_description/urdf/robotino.urdf.xacro (robot description, xacro)
@@ -108,9 +108,4 @@
     </collision>
   </link>
-  <!--joint name="platform_to_camera_base" type="fixed">
-    <parent link="platform_link"/>
-    <child link="camera_base_link"/>
-    <origin xyz="0.17 0 0.09" rpy="0 0 0"/>
-  </joint-->
   <joint name="camera_tilt_joint" type="revolute">
     <parent link="platform_link"/>
@@ -125,5 +120,4 @@
       mesh_package="manipulator_description"
       xyz="0.18 -0.115 0.0"
-      rpy="0 0 1.5707"
-  />
+      rpy="0 0 1.5707"/>
 </robot>
