Commit message: purge

File: PC_user/src/Hardware/robotino/robotino_description/urdf/robotino.urdf.xacro (robot description, xacro)
@@ -1,5 +1,5 @@
 <?xml version="1.0"?>
 <robot xmlns:xacro="http://www.ros.org/wiki/xacro" name="robotino">
-  <xacro:include filename="$(find manipulator_description)/urdf/manipulator.urdf.xacro" />
+  <xacro:include filename="$(find xarm_description)/urdf/xarm6/xarm6.urdf.xacro"/>
   <!-- ******************** Properties ******************** -->
   <xacro:property name="mesh_scale" value="0.01 0.01 0.01"/>
@@ -116,11 +116,33 @@
   <limit lower="${-0.541}" upper="${0.541}" effort="1.0" velocity="1.0"/>
 </joint>
-  <!-- ***************** Manipulator ****************-->
-  <xacro:prismatic_manipulator
-    prefix="manipulator_"
-    parent_link="platform_link"
-    mesh_package="manipulator_description"
-    xyz="0.0 0.0 0.0"
-    rpy="0 0 1.570796"
+<!-- ***************** Manipulator ****************-->
+  <xacro:property name="use_xacro_load_yaml" value="false"/>
+  <xacro:xarm6_urdf
+    prefix="xarm_"
   />
+  <!-- Fixed joint between robotino and arm base -->
+  <joint name="robotino_to_xarm_mount" type="fixed">
+    <parent link="platform_link"/>
+    <child link="xarm_link0"/>
+    <origin xyz="0 0 0.35" rpy="0 0 0"/> <!-- Ajusta la altura según montaje real -->
+  </joint>
+<!--<xacro:property name="is_ros2" value="false"/>
+<xacro:property name="use_xacro_load_yaml" value="false"/>
+<xacro:include filename="$(find xarm_description)/urdf/common/common.link.xacro" />
+<xacro:common_link_visual mesh_path="$(find xarm_description)/meshes/xarm6" />
+ <xacro:xarm6_robot
+    prefix="xarm_"
+    limited="false"
+    velocity_control="false"
+    add_gripper="false"
+    add_bio_gripper="false"
+    model_num="0"
+    inertial_params_filename=""
+    kinematics_params_filename=""
+  />
+  <joint name="platform_to_xarm" type="fixed">
+    <parent link="platform_link"/>
+    <child link="xarm_link_base"/>
+    <origin xyz="0 0 0" rpy="0 0 0"/>
+  </joint>-->
 </robot>

Commit message: add xarm in .xacro

File: PC_user/src/Hardware/robotino/robotino_description/urdf/robotino.urdf.xacro (robot description, xacro)
@@ -1,6 +1,8 @@
 <?xml version="1.0"?>
 <robot xmlns:xacro="http://www.ros.org/wiki/xacro" name="robotino">
+  <!-- ==================== Includes ==================== -->
   <xacro:include filename="$(find xarm_description)/urdf/xarm6/xarm6.urdf.xacro"/>
-  <!-- ******************** Properties ******************** -->
+  <xacro:include filename="$(find xarm_description)/urdf/xarm_device_macro.xacro" />
+  <!-- ==================== Properties ==================== -->
   <xacro:property name="mesh_scale" value="0.01 0.01 0.01"/>
   <xacro:property name="wheel_mesh" value="package://robotino_description/model/Robotino3_SplitWheel.dae"/>
@@ -9,5 +11,5 @@
   <xacro:property name="hokuyo_mesh" value="package://robotino_description/meshes/sensors/hokuyo.dae"/>
   <xacro:property name="kinect_mesh" value="package://robotino_description/meshes/sensors/kinect.dae"/>
-  <!-- ******************** Macros ******************** -->
+  <!-- ==================== Macros ==================== -->
   <xacro:macro name="wheel_link" params="index xyz rpy">
     <link name="wheel${index}_link">
@@ -32,5 +34,5 @@
     </joint>
   </xacro:macro>
-  <!-- ******************** Base ******************** -->
+  <!-- ==================== Base ==================== -->
   <link name="base_link">
     <visual>
@@ -47,12 +49,12 @@
     </collision>
   </link>
-  <!-- ******************** Wheel ******************** -->
+  <!-- ==================== Wheels ==================== -->
   <xacro:wheel_link index="0" xyz="-0.1825 -0.0001 0.059154" rpy="0 0 1.570796"/>
   <xacro:wheel_link index="1" xyz="0.090625 -0.157067 0.059154" rpy="0 0 3.665191"/>
   <xacro:wheel_link index="2" xyz="0.090625 0.156867 0.059154" rpy="0 0 -0.523599"/>
-  <!-- ******************** Tower ******************** -->
-  <link name="tower_link">
+  <!-- ==================== Tower (Platform) ==================== -->
+  <link name="platform_link">
     <visual>
-      <origin xyz="0 0 0" rpy="0 0 0"/>
+      <origin xyz="0 0 -0.70" rpy="0 0 1.5707"/>
       <geometry>
         <mesh filename="${tower_mesh}" scale="0.009 0.009 0.009"/>
@@ -60,17 +62,9 @@
     </visual>
     <collision>
-      <origin xyz="0 0 0" rpy="0 0 0"/>
+      <origin xyz="0 0 -0.70" rpy="0 0 1.5707"/>
       <geometry>
         <mesh filename="${tower_mesh}" scale="0.009 0.009 0.009"/>
       </geometry>
     </collision>
-  </link>
-  <joint name="tower_joint" type="fixed">
-    <parent link="base_link"/>
-    <child link="tower_link"/>
-    <origin xyz="0 0 0.06" rpy="0 0 1.5707"/>
-  </joint>
-  <!-- ******************** Platform link ******************** -->
-  <link name="platform_link">
   </link>
   <joint name="platform_joint" type="fixed">
@@ -79,5 +73,5 @@
     <origin xyz="0 0 0.76" rpy="0 0 0"/>
   </joint>
-  <!-- ******************** Hokuyo ******************** -->
+  <!-- ==================== Hokuyo Sensor ==================== -->
   <link name="laser_link">
     <visual>
@@ -87,4 +81,10 @@
       </geometry>
     </visual>
+    <collision>
+      <origin xyz="0 0 -0.055" rpy="0 0 1.57"/>
+      <geometry>
+        <mesh filename="${hokuyo_mesh}" scale="${mesh_scale}"/>
+      </geometry>
+    </collision>
   </link>
   <joint name="base_to_hokuyo" type="fixed">
@@ -93,56 +93,107 @@
     <origin xyz="0.07 0.0 0.28" rpy="0 0 0"/>
   </joint>
-  <!-- Soporte fijo del Kinect -->
-<link name="kinect_base_link"/>
-<joint name="platform_to_kinect_base" type="fixed">
-  <parent link="platform_link"/>
-  <child link="kinect_base_link"/>
-  <origin xyz="0.17 0 0.09" rpy="0 0 0"/>
-</joint>
-<!-- Eje móvil del motor del Kinect -->
-<link name="camera_link">
-  <visual>
-    <origin xyz="0 0 0" rpy="0 0 1.57"/>
-    <geometry>
-      <mesh filename="${kinect_mesh}" scale="1 1 1"/>
-    </geometry>
-  </visual>
-</link>
-<joint name="kinect_tilt_joint" type="revolute">
-  <parent link="kinect_base_link"/>
-  <child link="camera_link"/>
-  <origin xyz="0 0 0" rpy="0 0 0"/>
-  <axis xyz="0 1 0"/> <!-- eje de inclinación -->
-  <limit lower="${-0.541}" upper="${0.541}" effort="1.0" velocity="1.0"/>
-</joint>
-<!-- ***************** Manipulator ****************-->
-  <xacro:property name="use_xacro_load_yaml" value="false"/>
-  <xacro:xarm6_urdf
-    prefix="xarm_"
+  <!-- ==================== Kinect Sensor ==================== -->
+  <link name="camera_base_link"/>
+  <link name="camera_link">
+    <visual>
+      <origin xyz="0 0 0" rpy="0 0 1.57"/>
+      <geometry>
+        <mesh filename="${kinect_mesh}" scale="1 1 1"/>
+      </geometry>
+    </visual>
+  </link>
+  <joint name="platform_to_camera_base" type="fixed">
+    <parent link="platform_link"/>
+    <child link="camera_base_link"/>
+    <origin xyz="0.17 0 0.025" rpy="0 0 0"/>
+  </joint>
+  <joint name="camera_tilt_joint" type="revolute">
+    <parent link="camera_base_link"/>
+    <child link="camera_link"/>
+    <origin xyz="0 0 0" rpy="0 0 0"/>
+    <axis xyz="0 1 0"/>
+    <limit lower="${-0.541}" upper="${0.541}" effort="1.0" velocity="1.0"/>
+  </joint>
+  <!-- ==================== Manipulator (XArm) ==================== -->
+  <!-- XArm arguments -->
+  <xacro:arg name="prefix" default="arm_"/>
+  <xacro:arg name="hw_ns" default="xarm"/>
+  <xacro:arg name="limited" default="false"/>
+  <xacro:arg name="effort_control" default="false"/>
+  <xacro:arg name="velocity_control" default="false"/>
+  <xacro:arg name="add_gripper" default="false"/>
+  <xacro:arg name="add_vacuum_gripper" default="false"/>
+  <xacro:arg name="add_bio_gripper" default="false"/>
+  <xacro:arg name="model1300" default="false"/>
+  <xacro:arg name="dof" default="6"/>
+  <xacro:arg name="robot_ip" default="192.168.1.212"/>
+  <xacro:arg name="robot_type" default="xarm"/>
+  <xacro:arg name="robot_sn" default=""/>
+  <xacro:arg name="report_type" default="normal"/>
+  <xacro:arg name="ros2_control_plugin" default="uf_robot_hardware/UFRobotSystemHardware"/>
+  <xacro:arg name="ros2_control_params" default=""/>
+  <xacro:arg name="add_realsense_d435i" default="true"/>
+  <xacro:arg name="add_d435i_links" default="true"/>
+  <xacro:arg name="use_gazebo_camera" default="false"/>
+  <xacro:arg name="add_other_geometry" default="false"/>
+  <xacro:arg name="geometry_type" default="box"/>
+  <xacro:arg name="geometry_mass" default="0.1"/>
+  <xacro:arg name="geometry_height" default="0.1"/>
+  <xacro:arg name="geometry_radius" default="0.1"/>
+  <xacro:arg name="geometry_length" default="0.1"/>
+  <xacro:arg name="geometry_width" default="0.1"/>
+  <xacro:arg name="geometry_mesh_filename" default=""/>
+  <xacro:arg name="geometry_mesh_origin_xyz" default="0 0 0"/>
+  <xacro:arg name="geometry_mesh_origin_rpy" default="0 0 0"/>
+  <xacro:arg name="geometry_mesh_tcp_xyz" default="0 0 0"/>
+  <xacro:arg name="geometry_mesh_tcp_rpy" default="0 0 0"/>
+  <xacro:arg name="baud_checkset" default="true"/>
+  <xacro:arg name="default_gripper_baud" default="2000000"/>
+  <xacro:arg name="attach_to" default="platform_link"/>
+  <xacro:arg name="attach_xyz" default="-0.06 0 0.0"/>
+  <xacro:arg name="attach_rpy" default="0 0 0"/>
+  <xacro:arg name="mesh_suffix" default="stl"/>
+  <xacro:arg name="kinematics_suffix" default=""/>
+  <!-- Load XArm device -->
+  <xacro:xarm_device
+    prefix="$(arg prefix)"
+    hw_ns="$(arg hw_ns)"
+    limited="$(arg limited)"
+    effort_control="$(arg effort_control)"
+    velocity_control="$(arg velocity_control)"
+    add_gripper="$(arg add_gripper)"
+    add_vacuum_gripper="$(arg add_vacuum_gripper)"
+    add_bio_gripper="$(arg add_bio_gripper)"
+    dof="$(arg dof)"
+    ros2_control_plugin="$(arg ros2_control_plugin)"
+    robot_type="$(arg robot_type)"
+    load_gazebo_plugin="true"
+    ros2_control_params="$(arg ros2_control_params)"
+    add_realsense_d435i="$(arg add_realsense_d435i)"
+    add_d435i_links="$(arg add_d435i_links)"
+    add_other_geometry="$(arg add_other_geometry)"
+    geometry_type="$(arg geometry_type)"
+    geometry_mass="$(arg geometry_mass)"
+    geometry_height="$(arg geometry_height)"
+    geometry_radius="$(arg geometry_radius)"
+    geometry_length="$(arg geometry_length)"
+    geometry_width="$(arg geometry_width)"
+    geometry_mesh_filename="$(arg geometry_mesh_filename)"
+    geometry_mesh_origin_xyz="$(arg geometry_mesh_origin_xyz)"
+    geometry_mesh_origin_rpy="$(arg geometry_mesh_origin_rpy)"
+    geometry_mesh_tcp_xyz="$(arg geometry_mesh_tcp_xyz)"
+    geometry_mesh_tcp_rpy="$(arg geometry_mesh_tcp_rpy)"
+    robot_ip="$(arg robot_ip)"
+    report_type="$(arg report_type)"
+    baud_checkset="$(arg baud_checkset)"
+    default_gripper_baud="$(arg default_gripper_baud)"
+    model1300="$(arg model1300)"
+    attach_to="$(arg attach_to)"
+    attach_xyz="$(arg attach_xyz)"
+    attach_rpy="$(arg attach_rpy)"
+    robot_sn="$(arg robot_sn)"
+    use_gazebo_camera="$(arg use_gazebo_camera)"
+    mesh_suffix="$(arg mesh_suffix)"
+    kinematics_suffix="$(arg kinematics_suffix)"
   />
-  <!-- Fixed joint between robotino and arm base -->
-  <joint name="robotino_to_xarm_mount" type="fixed">
-    <parent link="platform_link"/>
-    <child link="xarm_link0"/>
-    <origin xyz="0 0 0.35" rpy="0 0 0"/> <!-- Ajusta la altura según montaje real -->
-  </joint>
-<!--<xacro:property name="is_ros2" value="false"/>
-<xacro:property name="use_xacro_load_yaml" value="false"/>
-<xacro:include filename="$(find xarm_description)/urdf/common/common.link.xacro" />
-<xacro:common_link_visual mesh_path="$(find xarm_description)/meshes/xarm6" />
- <xacro:xarm6_robot
-    prefix="xarm_"
-    limited="false"
-    velocity_control="false"
-    add_gripper="false"
-    add_bio_gripper="false"
-    model_num="0"
-    inertial_params_filename=""
-    kinematics_params_filename=""
-  />
-  <joint name="platform_to_xarm" type="fixed">
-    <parent link="platform_link"/>
-    <child link="xarm_link_base"/>
-    <origin xyz="0 0 0" rpy="0 0 0"/>
-  </joint>-->
 </robot>

Commit message: update URDF

File: PC_user/src/Hardware/robotino/robotino_description/urdf/robotino.urdf.xacro (robot description, xacro)
@@ -1,6 +1,7 @@
 <?xml version="1.0"?>
-<robot xmlns:xacro="http://www.ros.org/wiki/xacro" name="robotino">
+<robot xmlns:xacro="http://www.ros.org/wiki/xacro" name="robotino3">
+  <!-- ==================== Includes ==================== -->
   <xacro:include filename="$(find manipulator_description)/urdf/manipulator.urdf.xacro" />
-  <!-- ******************** Properties ******************** -->
+  <!-- ==================== Properties ==================== -->
   <xacro:property name="mesh_scale" value="0.01 0.01 0.01"/>
   <xacro:property name="wheel_mesh" value="package://robotino_description/model/Robotino3_SplitWheel.dae"/>
@@ -9,5 +10,5 @@
   <xacro:property name="hokuyo_mesh" value="package://robotino_description/meshes/sensors/hokuyo.dae"/>
   <xacro:property name="kinect_mesh" value="package://robotino_description/meshes/sensors/kinect.dae"/>
-  <!-- ******************** Macros ******************** -->
+  <!-- ==================== Macros ==================== -->
   <xacro:macro name="wheel_link" params="index xyz rpy">
     <link name="wheel${index}_link">
@@ -32,5 +33,5 @@
     </joint>
   </xacro:macro>
-  <!-- ******************** Base ******************** -->
+  <!-- ==================== Base ==================== -->
   <link name="base_link">
     <visual>
@@ -47,12 +48,12 @@
     </collision>
   </link>
-  <!-- ******************** Wheel ******************** -->
+  <!-- ==================== Wheels ==================== -->
   <xacro:wheel_link index="0" xyz="-0.1825 -0.0001 0.059154" rpy="0 0 1.570796"/>
   <xacro:wheel_link index="1" xyz="0.090625 -0.157067 0.059154" rpy="0 0 3.665191"/>
   <xacro:wheel_link index="2" xyz="0.090625 0.156867 0.059154" rpy="0 0 -0.523599"/>
-  <!-- ******************** Tower ******************** -->
-  <link name="tower_link">
+  <!-- ==================== Tower (Platform) ==================== -->
+  <link name="platform_link">
     <visual>
-      <origin xyz="0 0 0" rpy="0 0 0"/>
+      <origin xyz="0 0 -0.70" rpy="0 0 1.5707"/>
       <geometry>
         <mesh filename="${tower_mesh}" scale="0.009 0.009 0.009"/>
@@ -60,17 +61,9 @@
     </visual>
     <collision>
-      <origin xyz="0 0 0" rpy="0 0 0"/>
+      <origin xyz="0 0 -0.70" rpy="0 0 1.5707"/>
       <geometry>
         <mesh filename="${tower_mesh}" scale="0.009 0.009 0.009"/>
       </geometry>
     </collision>
-  </link>
-  <joint name="tower_joint" type="fixed">
-    <parent link="base_link"/>
-    <child link="tower_link"/>
-    <origin xyz="0 0 0.06" rpy="0 0 1.5707"/>
-  </joint>
-  <!-- ******************** Platform link ******************** -->
-  <link name="platform_link">
   </link>
   <joint name="platform_joint" type="fixed">
@@ -79,5 +72,5 @@
     <origin xyz="0 0 0.76" rpy="0 0 0"/>
   </joint>
-  <!-- ******************** Hokuyo ******************** -->
+  <!-- ==================== Hokuyo Sensor ==================== -->
   <link name="laser_link">
     <visual>
@@ -87,4 +80,10 @@
       </geometry>
     </visual>
+    <collision>
+      <origin xyz="0 0 -0.055" rpy="0 0 1.57"/>
+      <geometry>
+        <mesh filename="${hokuyo_mesh}" scale="${mesh_scale}"/>
+      </geometry>
+    </collision>
   </link>
   <joint name="base_to_hokuyo" type="fixed">
@@ -93,34 +92,33 @@
     <origin xyz="0.07 0.0 0.28" rpy="0 0 0"/>
   </joint>
-  <!-- Soporte fijo del Kinect -->
-<link name="kinect_base_link"/>
-<joint name="platform_to_kinect_base" type="fixed">
-  <parent link="platform_link"/>
-  <child link="kinect_base_link"/>
-  <origin xyz="0.17 0 0.09" rpy="0 0 0"/>
-</joint>
-<!-- Eje móvil del motor del Kinect -->
-<link name="camera_link">
-  <visual>
-    <origin xyz="0 0 0" rpy="0 0 1.57"/>
-    <geometry>
-      <mesh filename="${kinect_mesh}" scale="1 1 1"/>
-    </geometry>
-  </visual>
-</link>
-<joint name="kinect_tilt_joint" type="revolute">
-  <parent link="kinect_base_link"/>
-  <child link="camera_link"/>
-  <origin xyz="0 0 0" rpy="0 0 0"/>
-  <axis xyz="0 1 0"/> <!-- eje de inclinación -->
-  <limit lower="${-0.541}" upper="${0.541}" effort="1.0" velocity="1.0"/>
-</joint>
-  <!-- ***************** Manipulator ****************-->
+  <!-- ==================== Kinect Sensor ==================== -->
+  <link name="camera_base_link"/>
+  <link name="camera_link">
+    <visual>
+      <origin xyz="0 0 0" rpy="0 0 1.57"/>
+      <geometry>
+        <mesh filename="${kinect_mesh}" scale="1 1 1"/>
+      </geometry>
+    </visual>
+  </link>
+  <joint name="platform_to_camera_base" type="fixed">
+    <parent link="platform_link"/>
+    <child link="camera_base_link"/>
+    <origin xyz="0.17 0 0.09" rpy="0 0 0"/>
+  </joint>
+  <joint name="camera_tilt_joint" type="revolute">
+    <parent link="camera_base_link"/>
+    <child link="camera_link"/>
+    <origin xyz="0 0 0" rpy="0 0 0"/>
+    <axis xyz="0 1 0"/>
+    <limit lower="${-0.541}" upper="${0.541}" effort="1.0" velocity="1.0"/>
+  </joint>
+  <!-- ==================== Manipulator (Prismatic) ==================== -->
   <xacro:prismatic_manipulator
-    prefix="manipulator_"
-    parent_link="platform_link"
-    mesh_package="manipulator_description"
-    xyz="0.0 0.0 0.0"
-    rpy="0 0 1.570796"
+      prefix="manipulator_"
+      parent_link="platform_link"
+      mesh_package="manipulator_description"
+      xyz="0.0 0.0 0.0"
+      rpy="0 0 1.570796"
   />
 </robot>

Commit message: Setting for xarm and moveit

File: PC_user/src/Hardware/robotino/robotino_description/urdf/robotino.urdf.xacro (robot description, xacro)
@@ -1,3 +1,7 @@
 <?xml version="1.0"?>
+<!-- ==================================================================== -->
+<!-- ==================== ROBOTINO 4 - FestXarmKeshi ==================== -->
+<!-- ==================== PUMAS - Biorobotics Lab    ==================== -->
+<!-- ==================================================================== -->
 <robot xmlns:xacro="http://www.ros.org/wiki/xacro" name="robotino">
   <!-- ==================== Includes ==================== -->
@@ -8,5 +12,5 @@
   <xacro:property name="wheel_mesh" value="package://robotino_description/model/Robotino3_SplitWheel.dae"/>
   <xacro:property name="body_mesh" value="package://robotino_description/model/Robotino3_SplitMain_NoCamera.dae"/>
-  <xacro:property name="tower_mesh" value="package://robotino_description/model/Robotino3_Platform.dae"/>
+  <xacro:property name="tower_mesh" value="package://robotino_description/model/Robotino3_Platform-xarm.dae"/>
   <xacro:property name="hokuyo_mesh" value="package://robotino_description/meshes/sensors/hokuyo.dae"/>
   <xacro:property name="kinect_mesh" value="package://robotino_description/meshes/sensors/kinect.dae"/>
@@ -71,5 +75,5 @@
     <parent link="base_link"/>
     <child link="platform_link"/>
-    <origin xyz="0 0 0.76" rpy="0 0 0"/>
+    <origin xyz="0 0 0.57" rpy="0 0 0"/>
   </joint>
   <!-- ==================== Hokuyo Sensor ==================== -->
@@ -92,26 +96,4 @@
     <child link="laser_link"/>
     <origin xyz="0.07 0.0 0.28" rpy="0 0 0"/>
-  </joint>
-  <!-- ==================== Kinect Sensor ==================== -->
-  <link name="camera_base_link"/>
-  <link name="camera_link">
-    <visual>
-      <origin xyz="0 0 0" rpy="0 0 1.57"/>
-      <geometry>
-        <mesh filename="${kinect_mesh}" scale="1 1 1"/>
-      </geometry>
-    </visual>
-  </link>
-  <joint name="platform_to_camera_base" type="fixed">
-    <parent link="platform_link"/>
-    <child link="camera_base_link"/>
-    <origin xyz="0.17 0 0.025" rpy="0 0 0"/>
-  </joint>
-  <joint name="camera_tilt_joint" type="revolute">
-    <parent link="camera_base_link"/>
-    <child link="camera_link"/>
-    <origin xyz="0 0 0" rpy="0 0 0"/>
-    <axis xyz="0 1 0"/>
-    <limit lower="${-0.541}" upper="${0.541}" effort="1.0" velocity="1.0"/>
   </joint>
   <!-- ==================== Manipulator (XArm) ==================== -->
@@ -133,6 +115,6 @@
   <xacro:arg name="ros2_control_plugin" default="uf_robot_hardware/UFRobotSystemHardware"/>
   <xacro:arg name="ros2_control_params" default=""/>
-  <xacro:arg name="add_realsense_d435i" default="true"/>
-  <xacro:arg name="add_d435i_links" default="true"/>
+  <xacro:arg name="add_realsense_d435i" default="false"/>
+  <xacro:arg name="add_d435i_links" default="false"/>
   <xacro:arg name="use_gazebo_camera" default="false"/>
   <xacro:arg name="add_other_geometry" default="false"/>
@@ -151,5 +133,5 @@
   <xacro:arg name="default_gripper_baud" default="2000000"/>
   <xacro:arg name="attach_to" default="platform_link"/>
-  <xacro:arg name="attach_xyz" default="-0.06 0 0.0"/>
+  <xacro:arg name="attach_xyz" default="0.0 0.0 0.0"/>
   <xacro:arg name="attach_rpy" default="0 0 0"/>
   <xacro:arg name="mesh_suffix" default="stl"/>
@@ -197,3 +179,23 @@
     kinematics_suffix="$(arg kinematics_suffix)"
   />
+  <!-- ==================== Kinect Sensor ==================== -->
+  <link name="camera_link">
+    <visual>
+      <origin xyz="0 0 0" rpy="0 0 1.57"/>
+      <geometry>
+        <mesh filename="${kinect_mesh}" scale="1 1 1"/>
+      </geometry>
+    </visual>
+    <collision>
+      <origin xyz="0 0 0" rpy="0 0 1.57"/>
+      <geometry>
+        <mesh filename="${kinect_mesh}" scale="1 1 1"/>
+      </geometry>
+    </collision>
+  </link>
+  <joint name="platform_to_camera_link" type="fixed">
+    <parent link="arm_link6"/>
+    <child link="camera_link"/>
+    <origin xyz="0.08 0 -0.05" rpy="3.1415 -1.5707 0"/>
+  </joint>
 </robot>

Commit message: add config for xarm and moveit

File: PC_user/src/Hardware/robotino/robotino_description/urdf/robotino.urdf.xacro (robot description, xacro)
@@ -75,5 +75,5 @@
     <parent link="base_link"/>
     <child link="platform_link"/>
-    <origin xyz="0 0 0.57" rpy="0 0 0"/>
+    <origin xyz="0 0 0.455" rpy="0 0 0"/>
   </joint>
   <!-- ==================== Hokuyo Sensor ==================== -->
@@ -99,5 +99,5 @@
   <!-- ==================== Manipulator (XArm) ==================== -->
   <!-- XArm arguments -->
-  <xacro:arg name="prefix" default="arm_"/>
+  <xacro:arg name="prefix" default=""/>
   <xacro:arg name="hw_ns" default="xarm"/>
   <xacro:arg name="limited" default="false"/>
@@ -195,7 +195,7 @@
   </link>
   <joint name="platform_to_camera_link" type="fixed">
-    <parent link="arm_link6"/>
+    <parent link="link5"/>
     <child link="camera_link"/>
-    <origin xyz="0.08 0 -0.05" rpy="3.1415 -1.5707 0"/>
+    <origin xyz="0.15 0.035 0.0" rpy="1.5707 0 1.5707"/>
   </joint>
 </robot>
