Commit message: update urdf

File: PC_user/src/Hardware/robotino/robotino_description/urdf/robotino.urdf.xacro (robot description, xacro)
@@ -14,5 +14,5 @@
   <xacro:property name="tower_mesh" value="package://robotino_description/model/Robotino3_Platform-xarm.dae"/>
   <xacro:property name="hokuyo_mesh" value="package://robotino_description/meshes/sensors/hokuyo.dae"/>
-  <xacro:property name="kinect_mesh" value="package://robotino_description/meshes/sensors/kinect.dae"/>
+  <xacro:property name="kinect_mesh" value="package://robotino_description/meshes/sensors/kinect_without_base.dae"/>
   <!-- ==================== Macros ==================== -->
   <xacro:macro name="wheel_link" params="index xyz rpy">
@@ -109,5 +109,5 @@
   <xacro:arg name="model1300" default="false"/>
   <xacro:arg name="dof" default="6"/>
-  <xacro:arg name="robot_ip" default="192.168.1.212"/>
+  <xacro:arg name="robot_ip" default="172.27.1.212"/>
   <xacro:arg name="robot_type" default="xarm"/>
   <xacro:arg name="robot_sn" default=""/>
@@ -134,5 +134,5 @@
   <xacro:arg name="attach_to" default="platform_link"/>
   <xacro:arg name="attach_xyz" default="0.0 0.0 0.0"/>
-  <xacro:arg name="attach_rpy" default="0 0 0"/>
+  <xacro:arg name="attach_rpy" default="0 0 -1.047"/>
   <xacro:arg name="mesh_suffix" default="stl"/>
   <xacro:arg name="kinematics_suffix" default=""/>
@@ -197,5 +197,5 @@
     <parent link="link5"/>
     <child link="camera_link"/>
-    <origin xyz="0.15 0.035 0.0" rpy="1.5707 0 1.5707"/>
+    <origin xyz="0.12 0.035 0.0" rpy="1.5707 0 1.5707"/>
   </joint>
 </robot>

Commit message: sab 05 julio

File: PC_user/src/Hardware/robotino/robotino_description/urdf/robotino.urdf.xacro (robot description, xacro)
@@ -93,5 +93,5 @@
   </joint>
   <!-- ==================== Kinect Sensor ==================== -->
-  <link name="camera_base_link"/>
+  <!--link name="camera_base_link"/-->
   <link name="camera_link">
     <visual>
@@ -101,14 +101,20 @@
       </geometry>
     </visual>
+     <collision>
+      <origin xyz="0 0 0" rpy="0 0 1.57"/>
+      <geometry>
+        <mesh filename="${kinect_mesh}" scale="1 1 1"/>
+      </geometry>
+    </collision>
   </link>
-  <joint name="platform_to_camera_base" type="fixed">
+  <!--joint name="platform_to_camera_base" type="fixed">
     <parent link="platform_link"/>
     <child link="camera_base_link"/>
     <origin xyz="0.17 0 0.09" rpy="0 0 0"/>
-  </joint>
+  </joint-->
   <joint name="camera_tilt_joint" type="revolute">
-    <parent link="camera_base_link"/>
+    <parent link="platform_link"/>
     <child link="camera_link"/>
-    <origin xyz="0 0 0" rpy="0 0 0"/>
+    <origin xyz="0.17 0 0.095" rpy="0 0 0"/>
     <axis xyz="0 1 0"/>
     <limit lower="${-0.541}" upper="${0.541}" effort="1.0" velocity="1.0"/>

Commit message: update xacro

File: PC_user/src/Hardware/robotino/robotino_description/urdf/robotino.urdf.xacro (robot description, xacro)
@@ -125,6 +125,6 @@
       parent_link="platform_link"
       mesh_package="manipulator_description"
-      xyz="0.0 0.0 0.0"
-      rpy="0 0 1.570796"
+      xyz="0.18 -0.115 0.0"
+      rpy="0 0 1.5707"
   />
 </robot>

File: Robotino/src/manipulator/manipulator_description/urdf/manipulador_ajustes.urdf (robot description, URDF)
Before this commit: robot Manipulator, 7 links, 7 joints
Links:
- added link AluminumBase_link; collision mesh filename=package://manipulator_description/meshes/AluminumBase.stl scale=0.001 0.001 0.001; visual mesh filename=package://manipulator_description/meshes/AluminumBase.stl scale=0.001 0.001 0.001
Joints:
- joint AxisX_joint: axis 1 0 0 -> 0 1 0; limit lower=0 upper=0.105 effort=10.0 velocity=0.5 -> lower=-0.21592 upper=0.0 effort=10.0 velocity=0.5; origin xyz=0.02504 0.056 0.081 rpy=0 0 0 -> xyz=-0.00475 0.25696 0.02 rpy=0 0 0; parent AxisY_link -> BaseFrame_link
- joint AxisY_joint: axis 0 1 0 -> 1 0 0; limit lower=-0.21592 upper=0.0 effort=10.0 velocity=0.5 -> lower=0 upper=0.105 effort=10.0 velocity=0.5; origin xyz=-0.00475 0.25696 0.02 rpy=0 0 0 -> xyz=0.02504 0.056 0.081 rpy=0 0 0; parent BaseFrame_link -> AxisX_link
- joint AxisZ_joint: parent AxisX_link -> AxisY_link
- joint BaseFrame_joint: parent platform_link -> AluminumBase_link

Commit message: ultimos cambios, este es el chido

File: PC_user/src/Hardware/robotino/robotino_description/urdf/robotino.urdf.xacro (robot description, xacro)
@@ -108,10 +108,10 @@
     </collision>
   </link>
-  <joint name="camera_tilt_joint" type="revolute">
+  <joint name="camera_tilt_joint" type="fixed">
     <parent link="platform_link"/>
     <child link="camera_link"/>
-    <origin xyz="0.17 0 0.095" rpy="0 0 0"/>
-    <axis xyz="0 1 0"/>
-    <limit lower="${-0.541}" upper="${0.541}" effort="1.0" velocity="1.0"/>
+    <origin xyz="0.17 0 0.095" rpy="0 0.07 0"/>
+    <!--axis xyz="0 1 0"/-->
+    <!--limit lower="${-0.541}" upper="${0.541}" effort="1.0" velocity="1.0"/-->
   </joint>
   <!-- ==================== Manipulator (Prismatic) ==================== -->
